Commit message: added camera to robot

File: src/my_robot/urdf/my_robot.xacro (robot description, xacro)
@@ -63,5 +63,5 @@
         <origin xyz="0 0 0" rpy=" 0 1.5707 1.5707"/>
         <geometry>
-            <cylinder length="0.1" radius="0.05"/>
+            <cylinder length="0.05" radius="0.1"/>
         </geometry>
     </visual>
@@ -69,5 +69,5 @@
         <origin xyz="0 0 0" rpy=" 0 1.5707 1.5707"/>
         <geometry>
-            <cylinder length="0.1" radius="0.05"/>
+            <cylinder length="0.05" radius="0.1"/>
         </geometry>
     </collision>
@@ -108,3 +108,27 @@
     <dynamics damping="1.0" friction="1.0"/>
   </joint>
+  <link name="camera">
+    <inertial>
+      <mass value="0.1"/>
+      <origin xyz="0 0 0" rpy="0 0 0"/>
+      <inertia ixx="1e-6" ixy="0" ixz="0" iyy="1e-6" iyz="0" izz="1e-6"/>
+    </inertial>
+    <collision name="camera_collision">
+      <origin xyz="0 0 0" rpy="0 0 0"/>
+      <geometry>
+        <box size="0.05 0.05 0.05"/>
+      </geometry>
+    </collision>
+    <visual name="camera_visual">
+      <origin xyz="0 0 0" rpy="0 0 0"/>
+      <geometry>
+        <box size="0.05 0.05 0.05"/>
+      </geometry>
+    </visual>
+  </link>
+  <joint type="fixed" name="camera_joint">
+    <origin xyz="0.2 0 0"/>
+    <child link="camera"/>
+    <parent link="chassis"/>
+  </joint>
 </robot>

Commit message: added hokuyo lidar to robot

File: src/my_robot/urdf/my_robot.xacro (robot description, xacro)
@@ -132,3 +132,33 @@
     <parent link="chassis"/>
   </joint>
+  <link name="hokuyo">
+    <inertial>
+      <mass value="1e-5"/>
+      <origin xyz="0 0 0" rpy="0 0 0"/>
+      <inertia ixx="1e-6" ixy="0" ixz="0" iyy="1e-6" iyz="0" izz="1e-6"/>
+    </inertial>
+    <collision name="hokuyo_collision">
+      <origin xyz="0 0 0" rpy="0 0 0"/>
+      <geometry>
+        <box size="0.1 0.1 0.1"/>
+      </geometry>
+    </collision>
+    <visual>
+      <origin xyz="0 0 0" rpy="0 0 0"/>
+      <geometry>
+        <mesh filename="package://my_robot/meshes/hokuyo.dae"/>
+      </geometry>
+    </visual>
+  </link>
+  <joint type="fixed" name="hokuyo_joint">
+    <origin xyz="0.15 0 0.1"/>
+    <child link="hokuyo"/>
+    <parent link="chassis"/>
+  </joint>
+  <gazebo reference="left_wheel">
+    <material>Gazebo/Black</material>
+  </gazebo>
+  <gazebo reference="right_wheel">
+    <material>Gazebo/Black</material>
+  </gazebo>
 </robot>

Commit message: changed robot dimensions

File: src/my_robot/urdf/my_robot.xacro (robot description, xacro)
@@ -21,5 +21,5 @@
         <origin xyz="0 0 0" rpy=" 0 0 0"/>
         <geometry>
-            <box size=".4 .2 .1"/>
+            <box size=".6 .2 .1"/>
         </geometry>
     </collision>
@@ -27,5 +27,5 @@
         <origin xyz="0 0 0" rpy=" 0 0 0"/>
         <geometry>
-            <box size=".4 .2 .1"/>
+            <box size=".6 .2 .1"/>
         </geometry>
     </visual>
@@ -64,5 +64,5 @@
         <origin xyz="0 0 0" rpy=" 0 1.5707 1.5707"/>
         <geometry>
-            <cylinder length="0.05" radius="0.1"/>
+            <cylinder length="0.10" radius="0.1"/>
         </geometry>
     </visual>
@@ -70,5 +70,5 @@
         <origin xyz="0 0 0" rpy=" 0 1.5707 1.5707"/>
         <geometry>
-            <cylinder length="0.05" radius="0.1"/>
+            <cylinder length="0.10" radius="0.1"/>
         </geometry>
     </collision>
@@ -83,5 +83,5 @@
         <origin xyz="0 0 0" rpy=" 0 1.5707 1.5707"/>
         <geometry>
-            <cylinder length="0.05" radius="0.1"/>
+            <cylinder length="0.10" radius="0.1"/>
         </geometry>
     </visual>
@@ -89,5 +89,5 @@
         <origin xyz="0 0 0" rpy=" 0 1.5707 1.5707"/>
         <geometry>
-            <cylinder length="0.05" radius="0.1"/>
+            <cylinder length="0.10" radius="0.1"/>
         </geometry>
     </collision>
